File: AbacusPCB/AbacusPCB.kicad_pcb (KiCad board)
At the start: 2 copper layers, 263.5 x 76.2 mm, 134 parts, among them K1 KEYSW, K10 KEYSW, K11 KEYSW, K12 KEYSW, K13 KEYSW, K14 KEYSW, K15 KEYSW, K16 KEYSW, K17 KEYSW, K18 KEYSW, K19 KEYSW, K2 KEYSW, K20 KEYSW, K21 KEYSW, K22 KEYSW, K23 KEYSW, K24 KEYSW, K25 KEYSW, K26 KEYSW, K27 KEYSW, K28 KEYSW, K29 KEYSW, K3 KEYSW, K30 KEYSW, K31 KEYSW, K32 KEYSW, K33 KEYSW, K34 KEYSW, K35 KEYSW, K36 KEYSW, K37 KEYSW, K38 KEYSW, K39 KEYSW, K4 KEYSW, K40 KEYSW, K41 KEYSW, K42 KEYSW, K43 KEYSW, K44 KEYSW, K45 KEYSW, K5 KEYSW, K6 KEYSW, K7 KEYSW, K8 KEYSW, K9 KEYSW, SW1 Rotary_Encoder_Switch, SW2 SW_PUSH, U1 Elite-C_Pro-Micro

Commit message: gerbers sent
Parts:
- removed SW2: SW_PUSH, Button_Switch_THT:SW_PUSH_6mm
- added C17: 0.1uF, Capacitor_SMD:C_0603_1608Metric_Pad1.05x0.95mm_HandSolder, B.Cu at (100.0, 158.0)
- added D43: D, AbacusPCB:Diode, F.Cu at (292.1, 171.4)
- added G***: LOGO, AbacusPCB:art, B.Cu at (227.8, 146.1)
- added H11: MH, AbacusPCB:M3 Hole, F.Cu at (88.1, 112.7)
- added H12: MH, AbacusPCB:M3 Hole, F.Cu at (88.1, 181.0)
- added H13: MH, AbacusPCB:M3 Hole, F.Cu at (102.4, 181.0)
- added W17: WS2812B, AbacusPCB:WS2812_Hand_Solder, B.Cu at (95.2, 154.0)
- D1, D10, D11, D12, D13, D14, D15, D16, D17, D18, D19, D2, D20, D21, D22, D23, D24, D25, D26, D27, D28, D29, D3, D30, D31, D32, D33, D34, D35, D36, D37, D38, D39, D4, D40, D41, D42, D44, D45, D5, D6, D7, D8, D9: footprint Abacus_PCB:Diode -> AbacusPCB:Diode
- H1: moved to B.Cu
- SW1: footprint Rotary_Encoder:RotaryEncoder_Alps_EC11E-Switch_Vertical_H20mm -> AbacusPCB:Encoder
- moved H7 265.6 mm to (330.2, 165.9)
- moved H4 249.6 mm to (323.1, 145.3)
- moved H8 244.9 mm to (320.7, 123.8)
- moved H2 178.1 mm to (269.1, 175.4)
- moved H6 175.6 mm to (220.7, 175.4)
- moved C16 173.3 mm to (100.8, 173.0), turned to 0 degrees
- moved W16 169.3 mm to (95.2, 169.1), turned to 270 degrees
- moved W10 153.8 mm to (339.7, 165.9)
- moved W8 152.5 mm to (332.6, 127.8), turned to 180 degrees
- moved C15 145.0 mm to (124.6, 165.1), turned to 90 degrees
- moved W15 144.6 mm to (118.3, 165.9)
- moved C10 144.1 mm to (333.8, 166.6)
- moved C8 141.1 mm to (326.2, 128.5), turned to 90 degrees
- moved W9 136.1 mm to (335.0, 146.8), turned to 180 degrees
- moved W11 129.5 mm to (301.6, 165.9)
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Connections:
- U1 pad 10: /COL10 -> /COL7
- U1 pad 12: /COL8 -> /COL11
- U1 pad 13: /ROTS -> Net-(U1-Pad13)
- U1 pad 16: /ROTA -> /ROTB
- U1 pad 17: /ROTB -> /ROTA
- U1 pad 18: /COL7 -> /COL10
- U1 pad 19: /COL6 -> /COL8
- U1 pad 20: /COL5 -> /COL6
- U1 pad 6: /BUZZ -> /ROTS
- U1 pad 9: /COL11 -> /COL5
Routing:
- net /ROW3: track 0.00 -> 316.5 mm
- net /COL11: track 59.8 -> 320.3 mm
- net /COL10: track 62.5 -> 278.6 mm, vias 0 -> 1
- net /COL9: track 63.7 -> 275.2 mm, vias 0 -> 1
- net /COL8: track 61.4 -> 238.2 mm, vias 0 -> 1
- net /COL7: track 43.5 -> 217.1 mm, vias 0 -> 1
- net /COL6: track 62.9 -> 201.9 mm, vias 0 -> 1
- net /COL5: track 44.0 -> 180.0 mm, vias 0 -> 1
- net /COL4: track 43.5 -> 145.7 mm, vias 0 -> 1
- net /ROW2: track 198.6 -> 294.8 mm
- net /COL3: track 66.1 -> 149.7 mm, vias 0 -> 1
- net GND: track 0.00 -> 74.1 mm, vias 0 -> 33
- net /COL2: track 69.1 -> 134.1 mm, vias 0 -> 1
- net /ROW1: track 194.5 -> 258.3 mm
- net Net-(W11-Pad2): track 0.00 -> 52.5 mm
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- added copper zone on B.Cu, net +5V
- added copper zone on F.Cu, net GND
Other:
- board size 263.5 x 76.2 mm -> 265.1 x 76.2 mm
- board text added: "Rev 2"
- board text added: "https://github.com/nickolaij"

Commit message: finalisation changes for public release
Parts:
- moved C9 14.6 mm to (342.9, 144.5)
- turned W1 to 90 degrees
- turned W10 to 0 degrees
- turned W11 to 0 degrees
- turned W12 to 0 degrees
- turned W13 to 0 degrees
- turned W2 to 90 degrees
- turned W3 to 180 degrees
- turned W4 to 180 degrees
- turned W5 to 180 degrees
- turned W6 to 180 degrees
- turned W7 to 180 degrees
- turned W8 to 180 degrees
- turned W9 to 0 degrees
- renumbered W17 to W1, W8 to W10, W7 to W11, W6 to W12, W5 to W13, W4 to W14, W3 to W15, W2 to W16, W1 to W17, W16 to W2, W15 to W3, W14 to W4, W13 to W5, W12 to W6, W11 to W7, W10 to W8
Connections:
- W1 pad 1: GND -> +5V
- W1 pad 2: Net-(W17-Pad2) -> Net-(W1-Pad2)
- W1 pad 3: +5V -> GND
- W1 pad 4: Net-(W16-Pad2) -> /RGB
- W10 pad 1: GND -> +5V
- W10 pad 2: Net-(W8-Pad2) -> Net-(W10-Pad2)
- W10 pad 3: +5V -> GND
- W10 pad 4: Net-(W7-Pad2) -> Net-(W10-Pad4)
- W11 pad 1: GND -> +5V
- W11 pad 2: Net-(W7-Pad2) -> Net-(W11-Pad2)
- W11 pad 3: +5V -> GND
- W11 pad 4: Net-(W6-Pad2) -> Net-(W10-Pad2)
- W12 pad 1: GND -> +5V
- W12 pad 2: Net-(W6-Pad2) -> Net-(W12-Pad2)
- W12 pad 3: +5V -> GND
- W12 pad 4: Net-(W5-Pad2) -> Net-(W11-Pad2)
- W13 pad 1: GND -> +5V
- W13 pad 2: Net-(W5-Pad2) -> Net-(W13-Pad2)
- W13 pad 3: +5V -> GND
- W13 pad 4: Net-(W4-Pad2) -> Net-(W12-Pad2)
- W14 pad 2: Net-(W4-Pad2) -> Net-(W13-Pad2)
- W17 pad 4: /RGB -> Net-(W17-Pad4)
- W2 pad 1: GND -> +5V
- W2 pad 2: Net-(W16-Pad2) -> Net-(W2-Pad2)
- W2 pad 3: +5V -> GND
- W2 pad 4: Net-(W15-Pad2) -> Net-(W1-Pad2)
- W3 pad 1: GND -> +5V
- W3 pad 2: Net-(W15-Pad2) -> Net-(W3-Pad2)
- W3 pad 3: +5V -> GND
- W3 pad 4: Net-(W14-Pad2) -> Net-(W2-Pad2)
- W4 pad 1: GND -> +5V
- W4 pad 2: Net-(W14-Pad2) -> Net-(W4-Pad2)
- W4 pad 3: +5V -> GND
- W4 pad 4: Net-(W13-Pad2) -> Net-(W3-Pad2)
- W5 pad 1: GND -> +5V
- W5 pad 2: Net-(W13-Pad2) -> Net-(W5-Pad2)
- W5 pad 3: +5V -> GND
- W5 pad 4: Net-(W12-Pad2) -> Net-(W4-Pad2)
- W6 pad 1: GND -> +5V
- W6 pad 2: Net-(W12-Pad2) -> Net-(W6-Pad2)
- W6 pad 3: +5V -> GND
- W6 pad 4: Net-(W11-Pad2) -> Net-(W5-Pad2)
- W7 pad 1: GND -> +5V
- W7 pad 2: Net-(W11-Pad2) -> Net-(W7-Pad2)
- W7 pad 3: +5V -> GND
- W7 pad 4: Net-(W10-Pad2) -> Net-(W6-Pad2)
- W8 pad 1: GND -> +5V
- W8 pad 2: Net-(W10-Pad2) -> Net-(W8-Pad2)
- W8 pad 3: +5V -> GND
- W8 pad 4: Net-(W10-Pad4) -> Net-(W7-Pad2)
- W9 pad 1: GND -> +5V
- W9 pad 3: +5V -> GND
Routing:
- net Net-(W3-Pad2): track 0.00 -> 37.2 mm
- net Net-(W14-Pad2): track 37.2 -> 0.00 mm
- net Net-(W2-Pad2): track 0.00 -> 34.9 mm
- net Net-(W15-Pad2): track 34.9 -> 0.00 mm
- net Net-(W6-Pad2): track 33.1 -> 52.5 mm
- net Net-(W11-Pad2): track 52.5 -> 33.1 mm
- net Net-(W5-Pad2): track 33.1 -> 50.6 mm
- net Net-(W12-Pad2): track 50.6 -> 33.1 mm
- net /RGB: track 7.93 -> 25.0 mm, vias 0 -> 2
- net Net-(W16-Pad2): track 16.4 -> 0.00 mm
- net Net-(W1-Pad2): track 0.00 -> 16.4 mm
- net Net-(W7-Pad2): track 21.2 -> 34.0 mm
- net Net-(W10-Pad2): track 34.0 -> 21.2 mm
- net Net-(W8-Pad2): track 22.4 -> 28.4 mm
- net Net-(W10-Pad4): track 28.4 -> 22.4 mm
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