File: AbacusPCB/AbacusPCB.sch (KiCad schematic (older format))
At the start: 134 parts, among them K1 KEYSW, K10 KEYSW, K11 KEYSW, K12 KEYSW, K13 KEYSW, K14 KEYSW, K15 KEYSW, K16 KEYSW, K17 KEYSW, K18 KEYSW, K19 KEYSW, K2 KEYSW, K20 KEYSW, K21 KEYSW, K22 KEYSW, K23 KEYSW, K24 KEYSW, K25 KEYSW, K26 KEYSW, K27 KEYSW, K28 KEYSW, K29 KEYSW, K3 KEYSW, K30 KEYSW, K31 KEYSW, K32 KEYSW, K33 KEYSW, K34 KEYSW, K35 KEYSW, K36 KEYSW, K37 KEYSW, K38 KEYSW, K39 KEYSW, K4 KEYSW, K40 KEYSW, K41 KEYSW, K42 KEYSW, K43 KEYSW, K44 KEYSW, K45 KEYSW, K5 KEYSW, K6 KEYSW, K7 KEYSW, K8 KEYSW, K9 KEYSW, SW1 Rotary_Encoder_Switch, U1 Elite-C_Pro-Micro

Commit message: gerbers sent
Parts:
- added C17: 0.1uF, Capacitor_SMD:C_0603_1608Metric_Pad1.05x0.95mm_HandSolder, symbol Device:C
- added H11, H12, H13: MH, AbacusPCB:M3 Hole, symbol Mechanical:MountingHole
- added W17: WS2812B, AbacusPCB:WS2812_Hand_Solder, symbol LED:WS2812B
- D1, D10, D11, D12, D13, D14, D15, D16, D17, D18, D19, D2, D20, D21, D22, D23, D24, D25, D26, D27, D28, D29, D3, D30, D31, D32, D33, D34, D35, D36, D37, D38, D39, D4, D40, D41, D42, D43, D44, D45, D5, D6, D7, D8, D9: footprint Abacus_PCB:Diode -> AbacusPCB:Diode
- SW1: footprint Rotary_Encoder:RotaryEncoder_Alps_EC11E-Switch_Vertical_H20mm -> AbacusPCB:Encoder
Connections:
- net BUZZ is gone; now on net ROTS: U1.6 (D0/PWM)
- net +5V: now also C17.1, W17.3 (VSS)
- net COL10: now also U1.18 (B6/PWM); no longer U1.10 (E6)
- net COL11: now also U1.12 (B5/PWM); no longer U1.9 (D7/PWM)
- net COL5: now also U1.9 (D7/PWM); no longer U1.20 (B3/PWM)
- net COL6: now also U1.20 (B3/PWM); no longer U1.19 (B2)
- net COL7: now also U1.10 (E6); no longer U1.18 (B6/PWM)
- net COL8: now also U1.19 (B2); no longer U1.12 (B5/PWM)
- net GND: now also C17.2, W17.1 (VDD)
- net ROTA: now also U1.17; no longer U1.16
- net ROTB: now also U1.16; no longer U1.17
- net ROTS: no longer U1.13
- net at W16.2 (DOUT): now also W17.4 (DIN)
- no-connect marks 5 -> 6
Other:
- moved on the sheet: H1, H10, H2, H3, H4, H5, H6, H7, H8, H9

Commit message: finalisation changes for public release
Parts:
- renumbered W17 to W1, W8 to W10, W7 to W11, W6 to W12, W5 to W13, W4 to W14, W3 to W15, W2 to W16, W1 to W17, W16 to W2, W15 to W3, W14 to W4, W13 to W5, W12 to W6, W11 to W7, W10 to W8
Connections:
- net +5V: now also W1.1 (VDD), W10.1 (VDD), W11.1 (VDD), W12.1 (VDD), W13.1 (VDD), W2.1 (VDD), W3.1 (VDD), W4.1 (VDD), W5.1 (VDD), W6.1 (VDD), W7.1 (VDD), W8.1 (VDD), W9.1 (VDD); no longer W1.3 (VSS), W10.3 (VSS), W11.3 (VSS), W12.3 (VSS), W13.3 (VSS), W2.3 (VSS), W3.3 (VSS), W4.3 (VSS), W5.3 (VSS), W6.3 (VSS), W7.3 (VSS), W8.3 (VSS), W9.3 (VSS)
- net GND: now also W1.3 (VSS), W10.3 (VSS), W11.3 (VSS), W12.3 (VSS), W13.3 (VSS), W2.3 (VSS), W3.3 (VSS), W4.3 (VSS), W5.3 (VSS), W6.3 (VSS), W7.3 (VSS), W8.3 (VSS), W9.3 (VSS); no longer W1.1 (VDD), W10.1 (VDD), W11.1 (VDD), W12.1 (VDD), W13.1 (VDD), W2.1 (VDD), W3.1 (VDD), W4.1 (VDD), W5.1 (VDD), W6.1 (VDD), W7.1 (VDD), W8.1 (VDD), W9.1 (VDD)
- net RGB: now also W1.4 (DIN); no longer W17.4 (DIN)
- net at W14.2 (DOUT): now also W13.2 (DOUT); no longer W13.4 (DIN)
- net at W1.2 (DOUT): now also W2.4 (DIN)
- net at W2.2 (DOUT): now also W3.4 (DIN); no longer W1.4 (DIN)
- net at W12.4 (DIN): now also W11.2 (DOUT); no longer W13.2 (DOUT)
- net at W12.2 (DOUT): now also W13.4 (DIN); no longer W11.4 (DIN)
- net at W10.4 (DIN): now also W9.2 (DOUT); no longer W11.2 (DOUT)
- net at W10.2 (DOUT): now also W11.4 (DIN); no longer W9.4 (DIN)
- net at W8.4 (DIN): now also W7.2 (DOUT); no longer W9.2 (DOUT)
- net at W8.2 (DOUT): now also W9.4 (DIN); no longer W7.4 (DIN)
- net at W6.4 (DIN): now also W5.2 (DOUT); no longer W7.2 (DOUT)
- net at W6.2 (DOUT): now also W7.4 (DIN); no longer W5.4 (DIN)
- net at W4.4 (DIN): now also W3.2 (DOUT); no longer W5.2 (DOUT)
- net at W4.2 (DOUT): now also W5.4 (DIN); no longer W3.4 (DIN)
Changed lines of the file:
@@
 $EndComp
 $Comp
-L LED:WS2812B W1
+L LED:WS2812B W17
 U 1 1 5E28C5DF
 P 1350 4850
-F 0 "W1" V 1050 4950 50  0000 L CNN
+F 0 "W17" V 1050 4950 50  0000 L CNN
 F 1 "WS2812B" V 950 4950 50  0000 L CNN
 F 2 "AbacusPCB:WS2812_Hand_Solder" H 1400 4550 50  0001 L TNN
@@
 $EndComp
 $Comp
-L LED:WS2812B W2
+L LED:WS2812B W16
 U 1 1 5E2B0216
 P 1350 5600
-F 0 "W2" V 1050 5700 50  0000 L CNN
+F 0 "W16" V 1050 5700 50  0000 L CNN
 F 1 "WS2812B" V 950 5700 50  0000 L CNN
 F 2 "AbacusPCB:WS2812_Hand_Solder" H 1400 5300 50  0001 L TNN
@@
 $EndComp
 $Comp
-L LED:WS2812B W4
+L LED:WS2812B W14
 U 1 1 5E2E75A7
 P 1350 7100
-F 0 "W4" V 1050 7200 50  0000 L CNN
+F 0 "W14" V 1050 7200 50  0000 L CNN
 F 1 "WS2812B" V 950 7200 50  0000 L CNN
 F 2 "AbacusPCB:WS2812_Hand_Solder" H 1400 6800 50  0001 L TNN
@@
 Wire Wire Line
 	1350 4350 950  4350
-Text Label 950  4350 0    50   ~ 0
+Text Label 6500 7600 2    50   ~ 0
 RGB
 Text Label 8500 5150 0    50   ~ 0
@@
 	700  7100 950  7100
 $Comp
-L LED:WS2812B W5
+L LED:WS2812B W13
 U 1 1 5E4A1E21
 P 2650 4850
-F 0 "W5" V 2350 4950 50  0000 L CNN
-F 1 "WS2812B" V 2250 4950 50  0000 L CNN
+F 0 "W13" V 2250 4650 50  0000 L CNN
+F 1 "WS2812B" V 2350 4450 50  0000 L CNN
 F 2 "AbacusPCB:WS2812_Hand_Solder" H 2700 4550 50  0001 L TNN
 F 3 "https://cdn-shop.adafruit.com/datasheets/WS2812B.pdf" H 2750 4475 50  0001 L TNN
 	1    2650 4850
-	0    1    1    0
-$EndComp
-$Comp
-L LED:WS2812B W6
+	0    -1   -1   0
+$EndComp
+$Comp
+L LED:WS2812B W12
 U 1 1 5E4A1E27
 P 2650 5600
-F 0 "W6" V 2350 5700 50  0000 L CNN
-F 1 "WS2812B" V 2250 5700 50  0000 L CNN
+F 0 "W12" V 2250 5400 50  0000 L CNN
+F 1 "WS2812B" V 2350 5200 50  0000 L CNN
 F 2 "AbacusPCB:WS2812_Hand_Solder" H 2700 5300 50  0001 L TNN
 F 3 "https://cdn-shop.adafruit.com/datasheets/WS2812B.pdf" H 2750 5225 50  0001 L TNN
 	1    2650 5600
-	0    1    1    0
-$EndComp
-$Comp
-L LED:WS2812B W7
+	0    -1   -1   0
+$EndComp
+$Comp
+L LED:WS2812B W11
 U 1 1 5E4A1E2D
 P 2650 6350
-F 0 "W7" V 2350 6450 50  0000 L CNN
-F 1 "WS2812B" V 2250 6450 50  0000 L CNN
+F 0 "W11" V 2250 6150 50  0000 L CNN
+F 1 "WS2812B" V 2350 5950 50  0000 L CNN
 F 2 "AbacusPCB:WS2812_Hand_Solder" H 2700 6050 50  0001 L TNN
 F 3 "https://cdn-shop.adafruit.com/datasheets/WS2812B.pdf" H 2750 5975 50  0001 L TNN
 	1    2650 6350
-	0    1    1    0
-$EndComp
-$Comp
-L LED:WS2812B W8
+	0    -1   -1   0
+$EndComp
+$Comp
+L LED:WS2812B W10
 U 1 1 5E4A1E33
 P 2650 7100
-F 0 "W8" V 2350 7200 50  0000 L CNN
-F 1 "WS2812B" V 2250 7200 50  0000 L CNN
+F 0 "W10" V 2250 6900 50  0000 L CNN
+F 1 "WS2812B" V 2350 6700 50  0000 L CNN
 F 2 "AbacusPCB:WS2812_Hand_Solder" H 2700 6800 50  0001 L TNN
 F 3 "https://cdn-shop.adafruit.com/datasheets/WS2812B.pdf" H 2750 6725 50  0001 L TNN
 	1    2650 7100
-	0    1    1    0
+	0    -1   -1   0
 $EndComp
 Wire Wire Line
@@
 U 1 1 5E4DE106
 P 3950 4850
-F 0 "W9" V 3650 4950 50  0000 L CNN
-F 1 "WS2812B" V 3550 4950 50  0000 L CNN
+F 0 "W9" V 3550 4650 50  0000 L CNN
+F 1 "WS2812B" V 3650 4450 50  0000 L CNN
 F 2 "AbacusPCB:WS2812_Hand_Solder" H 4000 4550 50  0001 L TNN
 F 3 "https://cdn-shop.adafruit.com/datasheets/WS2812B.pdf" H 4050 4475 50  0001 L TNN
 	1    3950 4850
-	0    1    1    0
-$EndComp
-$Comp
-L LED:WS2812B W10
+	0    -1   -1   0
+$EndComp
+$Comp
+L LED:WS2812B W8
 U 1 1 5E4DE10C
 P 3950 5600
-F 0 "W10" V 3650 5700 50  0000 L CNN
-F 1 "WS2812B" V 3550 5700 50  0000 L CNN
+F 0 "W8" V 3550 5350 50  0000 L CNN
+F 1 "WS2812B" V 3650 5200 50  0000 L CNN
 F 2 "AbacusPCB:WS2812_Hand_Solder" H 4000 5300 50  0001 L TNN
 F 3 "https://cdn-shop.adafruit.com/datasheets/WS2812B.pdf" H 4050 5225 50  0001 L TNN
 	1    3950 5600
-	0    1    1    0
-$EndComp
-$Comp
-L LED:WS2812B W11
+	0    -1   -1   0
+$EndComp
+$Comp
+L LED:WS2812B W7
 U 1 1 5E4DE112
 P 3950 6350
-F 0 "W11" V 3650 6450 50  0000 L CNN
-F 1 "WS2812B" V 3550 6450 50  0000 L CNN
+F 0 "W7" V 3550 6100 50  0000 L CNN
+F 1 "WS2812B" V 3650 5950 50  0000 L CNN
 F 2 "AbacusPCB:WS2812_Hand_Solder" H 4000 6050 50  0001 L TNN
 F 3 "https://cdn-shop.adafruit.com/datasheets/WS2812B.pdf" H 4050 5975 50  0001 L TNN
 	1    3950 6350
-	0    1    1    0
-$EndComp
-$Comp
-L LED:WS2812B W12
+	0    -1   -1   0
+$EndComp
+$Comp
+L LED:WS2812B W6
 U 1 1 5E4DE118
 P 3950 7100
-F 0 "W12" V 3650 7200 50  0000 L CNN
-F 1 "WS2812B" V 3550 7200 50  0000 L CNN
+F 0 "W6" V 3550 6850 50  0000 L CNN
+F 1 "WS2812B" V 3650 6700 50  0000 L CNN
 F 2 "AbacusPCB:WS2812_Hand_Solder" H 4000 6800 50  0001 L TNN
 F 3 "https://cdn-shop.adafruit.com/datasheets/WS2812B.pdf" H 4050 6725 50  0001 L TNN
 	1    3950 7100
-	0    1    1    0
+	0    -1   -1   0
 $EndComp
 Wire Wire Line
@@
 	3300 7100 3550 7100
 $Comp
-L LED:WS2812B W13
+L LED:WS2812B W5
 U 1 1 5E50A3DE
 P 5250 4850
-F 0 "W13" V 4950 4950 50  0000 L CNN
-F 1 "WS2812B" V 4850 4950 50  0000 L CNN
+F 0 "W5" V 4850 4600 50  0000 L CNN
+F 1 "WS2812B" V 4950 4450 50  0000 L CNN
 F 2 "AbacusPCB:WS2812_Hand_Solder" H 5300 4550 50  0001 L TNN
 F 3 "https://cdn-shop.adafruit.com/datasheets/WS2812B.pdf" H 5350 4475 50  0001 L TNN
 	1    5250 4850
-	0    1    1    0
-$EndComp
-$Comp
-L LED:WS2812B W14
+	0    -1   -1   0
+$EndComp
+$Comp
+L LED:WS2812B W4
 U 1 1 5E50A3E4
 P 5250 5600
-F 0 "W14" V 4950 5700 50  0000 L CNN
-F 1 "WS2812B" V 4850 5700 50  0000 L CNN
+F 0 "W4" V 4850 5400 50  0000 L CNN
+F 1 "WS2812B" V 4950 5200 50  0000 L CNN
 F 2 "AbacusPCB:WS2812_Hand_Solder" H 5300 5300 50  0001 L TNN
 F 3 "https://cdn-shop.adafruit.com/datasheets/WS2812B.pdf" H 5350 5225 50  0001 L TNN
 	1    5250 5600
-	0    1    1    0
-$EndComp
-$Comp
-L LED:WS2812B W15
+	0    -1   -1   0
+$EndComp
+$Comp
+L LED:WS2812B W3
 U 1 1 5E50A3EA
 P 5250 6350
-F 0 "W15" V 4950 6450 50  0000 L CNN
-F 1 "WS2812B" V 4850 6450 50  0000 L CNN
+F 0 "W3" V 4850 6150 50  0000 L CNN
+F 1 "WS2812B" V 4950 5950 50  0000 L CNN
 F 2 "AbacusPCB:WS2812_Hand_Solder" H 5300 6050 50  0001 L TNN
 F 3 "https://cdn-shop.adafruit.com/datasheets/WS2812B.pdf" H 5350 5975 50  0001 L TNN
 	1    5250 6350
-	0    1    1    0
-$EndComp
-$Comp
-L LED:WS2812B W16
+	0    -1   -1   0
+$EndComp
+$Comp
+L LED:WS2812B W2
 U 1 1 5E50A3F0
 P 5250 7100
-F 0 "W16" V 4950 7200 50  0000 L CNN
-F 1 "WS2812B" V 4850 7200 50  0000 L CNN
+F 0 "W2" V 4850 6900 50  0000 L CNN
+F 1 "WS2812B" V 4950 6700 50  0000 L CNN
 F 2 "AbacusPCB:WS2812_Hand_Solder" H 5300 6800 50  0001 L TNN
 F 3 "https://cdn-shop.adafruit.com/datasheets/WS2812B.pdf" H 5350 6725 50  0001 L TNN
 	1    5250 7100
-	0    1    1    0
+	0    -1   -1   0
 $EndComp
 Wire Wire Line
@@
 $EndComp
 $Comp
-L LED:WS2812B W3
+L LED:WS2812B W15
 U 1 1 5E2C8E48
 P 1350 6350
-F 0 "W3" V 1050 6450 50  0000 L CNN
+F 0 "W15" V 1050 6450 50  0000 L CNN
 F 1 "WS2812B" V 950 6450 50  0000 L CNN
 F 2 "AbacusPCB:WS2812_Hand_Solder" H 1400 6050 50  0001 L TNN
@@
 $EndComp
 $Comp
-L LED:WS2812B W17
+L LED:WS2812B W1
 U 1 1 5E424024
 P 6500 7150
-F 0 "W17" V 6200 7250 50  0000 L CNN
-F 1 "WS2812B" V 6100 7250 50  0000 L CNN
+F 0 "W1" V 6100 6900 50  0000 L CNN
+F 1 "WS2812B" V 6200 6750 50  0000 L CNN
 F 2 "AbacusPCB:WS2812_Hand_Solder" H 6550 6850 50  0001 L TNN
 F 3 "https://cdn-shop.adafruit.com/datasheets/WS2812B.pdf" H 6600 6775 50  0001 L TNN
 	1    6500 7150
-	0    1    1    0
+	0    -1   -1   0
 $EndComp
 Wire Wire Line
@@
 Wire Wire Line
 	6500 6800 6500 6850
-NoConn ~ 6500 7600
+NoConn ~ 950  4350
 $EndSCHEMATC
